File: electronics/board_template/atmega328/template_atmega328p.brd (EAGLE design)
At the start: 48 x 48 mm, 42 parts, among them IC1 ATMEGA328P-MU, IC2 CP2104-F03-GMR, IC3 NCP1117ST50T3G, IC4 LMV358IDGKRG4, J1 GROVE_CONNECTOR2.0_1X4, J2 GROVE_CONNECTOR2.0_1X4, J3 10129383-906001ALF, J4 10129383-912001ALF, J5 10129383-912001ALF, Q1 FDN340P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

Commit message: Logo hinzugefügt
Parts:
- added U$1: LOGO_MORPHBOT5MM, topo-eng:LOGO_MORPHBOT
Changed lines of the file:
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@@
 <layer number="104" name="Name" color="7" fill="1" visible="no" active="yes"/>
 <layer number="116" name="Patch_BOT" color="9" fill="4" visible="no" active="yes"/>
+<layer number="120" name="brd_placement_notes" color="7" fill="1" visible="yes" active="yes"/>
 <layer number="121" name="_tsilk" color="7" fill="1" visible="no" active="yes"/>
 <layer number="122" name="_bsilk" color="7" fill="1" visible="no" active="yes"/>
+<layer number="144" name="DrillLegend" color="7" fill="1" visible="yes" active="yes"/>
+<layer number="145" name="DrillLegend_01-16" color="7" fill="1" visible="yes" active="yes"/>
+<layer number="146" name="DrillLegend_01-20" color="7" fill="1" visible="yes" active="yes"/>
 <layer number="151" name="HeatSink" color="14" fill="1" visible="no" active="no"/>
+<layer number="198" name="BMP198" color="7" fill="1" visible="yes" active="yes"/>
+<layer number="199" name="Contour" color="7" fill="1" visible="yes" active="yes"/>
 <layer number="200" name="200bmp" color="1" fill="10" visible="no" active="no"/>
 <layer number="201" name="201bmp" color="2" fill="1" visible="no" active="no"/>
@@
 <layer number="207" name="207bmp" color="15" fill="10" visible="no" active="no"/>
 <layer number="208" name="208bmp" color="9" fill="10" visible="no" active="yes"/>
+<layer number="209" name="Route9Document" color="7" fill="1" visible="yes" active="yes"/>
+<layer number="210" name="Route10Document" color="7" fill="1" visible="yes" active="yes"/>
+<layer number="211" name="Route11Document" color="7" fill="1" visible="yes" active="yes"/>
+<layer number="212" name="Route12Document" color="7" fill="1" visible="yes" active="yes"/>
+<layer number="213" name="Route13Document" color="7" fill="1" visible="yes" active="yes"/>
+<layer number="214" name="Route14Document" color="7" fill="1" visible="yes" active="yes"/>
+<layer number="215" name="Route15Document" color="7" fill="1" visible="yes" active="yes"/>
+<layer number="216" name="BottomDocument" color="7" fill="1" visible="yes" active="yes"/>
+<layer number="220" name="DimensionDocument" color="7" fill="1" visible="yes" active="yes"/>
+<layer number="221" name="tPlaceDocument" color="7" fill="1" visible="yes" active="yes"/>
+<layer number="222" name="bPlaceDocument" color="7" fill="1" visible="yes" active="yes"/>
+<layer number="225" name="tNamesDocument" color="7" fill="1" visible="yes" active="yes"/>
+<layer number="226" name="bNamesDocument" color="7" fill="1" visible="yes" active="yes"/>
+<layer number="227" name="tValuesDocument" color="7" fill="1" visible="yes" active="yes"/>
+<layer number="228" name="bValuesDocument" color="7" fill="1" visible="yes" active="yes"/>
+<layer number="229" name="tStopDocument" color="7" fill="1" visible="yes" active="yes"/>
+<layer number="230" name="bStopDocument" color="7" fill="1" visible="yes" active="yes"/>
+<layer number="231" name="tCreamDocument" color="7" fill="1" visible="yes" active="yes"/>
+<layer number="232" name="bCreamDocument" color="7" fill="1" visible="yes" active="yes"/>
+<layer number="233" name="tFinishDocument" color="7" fill="1" visible="yes" active="yes"/>
+<layer number="234" name="bFinishDocument" color="7" fill="1" visible="yes" active="yes"/>
+<layer number="235" name="tGlueDocument" color="7" fill="1" visible="yes" active="yes"/>
+<layer number="236" name="bGlueDocument" color="7" fill="1" visible="yes" active="yes"/>
+<layer number="244" name="DrillsDocument" color="7" fill="1" visible="yes" active="yes"/>
+<layer number="245" name="HolesDocument" color="7" fill="1" visible="yes" active="yes"/>
+<layer number="246" name="MillingDocument" color="7" fill="1" visible="yes" active="yes"/>
+<layer number="247" name="MeasuresDocument" color="7" fill="1" visible="yes" active="yes"/>
 <layer number="250" name="Descript" color="3" fill="1" visible="no" active="no"/>
 <layer number="251" name="SMDround" color="12" fill="11" visible="no" active="no"/>
@@
 <attribute name="VALUE" x="17.859015625" y="40.145653125" size="1.27" layer="27" rot="R270"/>
 </element>
+<element name="U$1" library="topo-eng" library_urn="urn:adsk.eagle:library:6646478" package="LOGO_MORPHBOT" value="LOGO_MORPHBOT5MM" x="46.630434375" y="1.122628125" smashed="yes" rot="R90"/>
 </elements>
 <signals>

Commit message: Fiducials eingefügt
Parts:
- added FID1, FID2, FID3: OPEN-PNP-FIDUCIAL, topo-eng:OPEN-PNP-FIDUCIAL
