File: electronics/board_template/atmega328/template_atmega328p.brd (EAGLE design)
At the start: 48 x 48 mm, 46 parts, among them IC1 ATMEGA328P-MU, IC2 CP2104-F03-GMR, IC3 NCP1117ST50T3G, IC4 LMV358IDGKRG4, J1 GROVE_CONNECTOR2.0_1X4, J2 GROVE_CONNECTOR2.0_1X4, J3 10129383-906001ALF, J4 10129383-912001ALF, J5 10129383-912001ALF, Q1 FDN340P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

Commit message: ESP32-Template: - USB-Datenleitungen getauscht (BugFix) 328P-Template: - USB-Datenleitungen getauscht (BugFix) - Reset-Leitung mit DTR verbunden (Zum Programieren über ARDUINO-IDE notwendig)
Parts:
- added C11: CL05B104KO5NNNC - 100n, rcl:C0402
Connections:
- new net DTR: C11.1, IC2.23
- net RESET: now also C11.2
- net USB_DN: now also D1.3, X1.2; no longer D1.4, X1.3
- net USB_DP: now also D1.4, X1.3; no longer D1.3, X1.2
Routing:
- net DTR: track 0.00 -> 33.7 mm, vias 0 -> 2
- net USB_DP: track 40.4 -> 34.7 mm, vias 0 -> 4
- net GND: track 212.4 -> 217.9 mm, vias 2 -> 3
- net RESET: track 45.8 -> 48.6 mm, vias 2 -> 3
- net USB_DN: track 40.2 -> 39.4 mm, vias 4 -> 2

Commit message: Logo geändert
Parts:
- IC3: device samacsys:SOT230P700X180-4N@1 -> samacsys:SOT230P700X180-4N
