File: electronics/board_template/atmega328/template_atmega328p.sch (EAGLE design)
At the start: 42 parts, among them IC1 ATMEGA328P-MU, IC2 CP2104-F03-GMR, IC3 NCP1117ST50T3G, IC4 LMV358IDGKRG4, J1 GROVE_CONNECTOR2.0_1X4, J2 GROVE_CONNECTOR2.0_1X4, J3 10129383-906001ALF, J4 10129383-912001ALF, J5 10129383-912001ALF, Q1 FDN340P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

Commit message: Logo hinzugefügt
Parts:
- added U$1: LOGO_MORPHBOT5MM, topo-eng:LOGO_MORPHBOT5MM
Changed lines of the file:
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@@
 <layer number="104" name="Name" color="7" fill="1" visible="no" active="yes"/>
 <layer number="116" name="Patch_BOT" color="9" fill="4" visible="no" active="yes"/>
+<layer number="120" name="brd_placement_notes" color="7" fill="1" visible="yes" active="yes"/>
 <layer number="121" name="_tsilk" color="7" fill="1" visible="no" active="yes"/>
 <layer number="122" name="_bsilk" color="7" fill="1" visible="no" active="yes"/>
+<layer number="144" name="DrillLegend" color="7" fill="1" visible="yes" active="yes"/>
+<layer number="145" name="DrillLegend_01-16" color="7" fill="1" visible="yes" active="yes"/>
+<layer number="146" name="DrillLegend_01-20" color="7" fill="1" visible="yes" active="yes"/>
 <layer number="151" name="HeatSink" color="14" fill="1" visible="no" active="no"/>
+<layer number="198" name="BMP198" color="7" fill="1" visible="yes" active="yes"/>
+<layer number="199" name="Contour" color="7" fill="1" visible="yes" active="yes"/>
 <layer number="200" name="200bmp" color="1" fill="10" visible="no" active="no"/>
 <layer number="201" name="201bmp" color="2" fill="1" visible="no" active="no"/>
@@
 <layer number="207" name="207bmp" color="15" fill="10" visible="no" active="no"/>
 <layer number="208" name="208bmp" color="9" fill="10" visible="no" active="yes"/>
+<layer number="209" name="Route9Document" color="7" fill="1" visible="yes" active="yes"/>
+<layer number="210" name="Route10Document" color="7" fill="1" visible="yes" active="yes"/>
+<layer number="211" name="Route11Document" color="7" fill="1" visible="yes" active="yes"/>
+<layer number="212" name="Route12Document" color="7" fill="1" visible="yes" active="yes"/>
+<layer number="213" name="Route13Document" color="7" fill="1" visible="yes" active="yes"/>
+<layer number="214" name="Route14Document" color="7" fill="1" visible="yes" active="yes"/>
+<layer number="215" name="Route15Document" color="7" fill="1" visible="yes" active="yes"/>
+<layer number="216" name="BottomDocument" color="7" fill="1" visible="yes" active="yes"/>
+<layer number="220" name="DimensionDocument" color="7" fill="1" visible="yes" active="yes"/>
+<layer number="221" name="tPlaceDocument" color="7" fill="1" visible="yes" active="yes"/>
+<layer number="222" name="bPlaceDocument" color="7" fill="1" visible="yes" active="yes"/>
+<layer number="225" name="tNamesDocument" color="7" fill="1" visible="yes" active="yes"/>
+<layer number="226" name="bNamesDocument" color="7" fill="1" visible="yes" active="yes"/>
+<layer number="227" name="tValuesDocument" color="7" fill="1" visible="yes" active="yes"/>
+<layer number="228" name="bValuesDocument" color="7" fill="1" visible="yes" active="yes"/>
+<layer number="229" name="tStopDocument" color="7" fill="1" visible="yes" active="yes"/>
+<layer number="230" name="bStopDocument" color="7" fill="1" visible="yes" active="yes"/>
+<layer number="231" name="tCreamDocument" color="7" fill="1" visible="yes" active="yes"/>
+<layer number="232" name="bCreamDocument" color="7" fill="1" visible="yes" active="yes"/>
+<layer number="233" name="tFinishDocument" color="7" fill="1" visible="yes" active="yes"/>
+<layer number="234" name="bFinishDocument" color="7" fill="1" visible="yes" active="yes"/>
+<layer number="235" name="tGlueDocument" color="7" fill="1" visible="yes" active="yes"/>
+<layer number="236" name="bGlueDocument" color="7" fill="1" visible="yes" active="yes"/>
+<layer number="244" name="DrillsDocument" color="7" fill="1" visible="yes" active="yes"/>
+<layer number="245" name="HolesDocument" color="7" fill="1" visible="yes" active="yes"/>
+<layer number="246" name="MillingDocument" color="7" fill="1" visible="yes" active="yes"/>
+<layer number="247" name="MeasuresDocument" color="7" fill="1" visible="yes" active="yes"/>
 <layer number="250" name="Descript" color="3" fill="1" visible="no" active="no"/>
 <layer number="251" name="SMDround" color="12" fill="11" visible="no" active="no"/>
@@
 <part name="R12" library="rcl" library_urn="urn:adsk.eagle:library:334" deviceset="R-EU_" device="R0402" package3d_urn="urn:adsk.eagle:package:23547/2" value="Uniroyal Elec 0402WGF1001TCE - 1k"/>
 <part name="R13" library="rcl" library_urn="urn:adsk.eagle:library:334" deviceset="R-EU_" device="R0402" package3d_urn="urn:adsk.eagle:package:23547/2" value="Uniroyal Elec 0402WGF6801TCE - 680R"/>
+<part name="U$1" library="topo-eng" library_urn="urn:adsk.eagle:library:6646478" deviceset="LOGO_MORPHBOT" device="5MM"/>
 </parts>
 <sheets>
@@
 <attribute name="VALUE" x="106.68" y="24.638" size="1.778" layer="96"/>
 </instance>
+<instance part="U$1" gate="G$1" x="68.58" y="66.04" smashed="yes"/>
 </instances>
 <busses>

Commit message: Fiducials eingefügt
Parts:
- added FID1, FID2, FID3: OPEN-PNP-FIDUCIAL, topo-eng:OPEN-PNP-FIDUCIAL
Changed lines of the file:
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@@
 <part name="R13" library="rcl" library_urn="urn:adsk.eagle:library:334" deviceset="R-EU_" device="R0402" package3d_urn="urn:adsk.eagle:package:23547/2" value="Uniroyal Elec 0402WGF6801TCE - 680R"/>
 <part name="U$1" library="topo-eng" library_urn="urn:adsk.eagle:library:6646478" deviceset="LOGO_MORPHBOT" device="5MM"/>
+<part name="FID1" library="topo-eng" library_urn="urn:adsk.eagle:library:6646478" deviceset="OPEN-PNP-FIDUCIAL" device=""/>
+<part name="FID2" library="topo-eng" library_urn="urn:adsk.eagle:library:6646478" deviceset="OPEN-PNP-FIDUCIAL" device=""/>
+<part name="FID3" library="topo-eng" library_urn="urn:adsk.eagle:library:6646478" deviceset="OPEN-PNP-FIDUCIAL" device=""/>
 </parts>
 <sheets>
@@
 </instance>
 <instance part="U$1" gate="G$1" x="68.58" y="66.04" smashed="yes"/>
+<instance part="FID1" gate="FID$1" x="93.98" y="48.26" smashed="yes">
+<attribute name="NAME" x="88.9" y="53.34" size="1.778" layer="94"/>
+</instance>
+<instance part="FID2" gate="FID$1" x="101.6" y="48.26" smashed="yes">
+<attribute name="NAME" x="96.52" y="53.34" size="1.778" layer="94"/>
+</instance>
+<instance part="FID3" gate="FID$1" x="109.22" y="48.26" smashed="yes">
+<attribute name="NAME" x="104.14" y="53.34" size="1.778" layer="94"/>
+</instance>
 </instances>
 <busses>

Commit message: ESP32-Template: - USB-Datenleitungen getauscht (BugFix) 328P-Template: - USB-Datenleitungen getauscht (BugFix) - Reset-Leitung mit DTR verbunden (Zum Programieren über ARDUINO-IDE notwendig)
Parts:
- added C11: CL05B104KO5NNNC - 100n, rcl:C-EUC0402
Connections:
- new net DTR: C11.1, IC2.DTR
- net RESET: now also C11.2
- net USB_DN: now also D1.K_2, X1G$1.2; no longer D1.K_3, X1G$1.3
- net USB_DP: now also D1.K_3, X1G$1.3; no longer D1.K_2, X1G$1.2
Changed lines of the file:
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@@
 <part name="FID2" library="topo-eng" library_urn="urn:adsk.eagle:library:6646478" deviceset="OPEN-PNP-FIDUCIAL" device=""/>
 <part name="FID3" library="topo-eng" library_urn="urn:adsk.eagle:library:6646478" deviceset="OPEN-PNP-FIDUCIAL" device=""/>
+<part name="C11" library="rcl" library_urn="urn:adsk.eagle:library:334" deviceset="C-EU" device="C0402" package3d_urn="urn:adsk.eagle:package:23626/1" value="CL05B104KO5NNNC - 100n"/>
 </parts>
 <sheets>
@@
 <attribute name="VALUE" x="165.1" y="128.778" size="1.778" layer="96"/>
 </instance>
+<instance part="C11" gate="G$1" x="144.78" y="121.92" smashed="yes" rot="R180">
+<attribute name="NAME" x="140.081" y="122.936" size="1.778" layer="95" rot="R270"/>
+<attribute name="VALUE" x="137.541" y="122.936" size="1.778" layer="96" rot="R270"/>
+</instance>
 </instances>
 <busses>
@@
 <net name="USB_DP" class="0">
 <segment>
+<pinref part="IC2" gate="G$1" pin="D+"/>
+<wire x1="129.54" y1="91.44" x2="121.92" y2="91.44" width="0.1524" layer="91"/>
+<label x="121.92" y="91.44" size="1.27" layer="95" ratio="5" rot="R180" xref="yes"/>
+</segment>
+<segment>
+<pinref part="X1" gate="G$1" pin="3"/>
+<wire x1="22.86" y1="25.4" x2="27.94" y2="25.4" width="0.1524" layer="91"/>
+<label x="27.94" y="25.4" size="1.27" layer="95" ratio="5" xref="yes"/>
+</segment>
+<segment>
+<pinref part="D1" gate="G$1" pin="K_3"/>
+<wire x1="86.36" y1="30.48" x2="88.9" y2="30.48" width="0.1524" layer="91"/>
+<label x="88.9" y="30.48" size="1.27" layer="95" ratio="5" xref="yes"/>
+</segment>
+</net>
+<net name="USB_DN" class="0">
+<segment>
+<pinref part="IC2" gate="G$1" pin="D-"/>
+<wire x1="129.54" y1="88.9" x2="121.92" y2="88.9" width="0.1524" layer="91"/>
+<label x="121.92" y="88.9" size="1.27" layer="95" ratio="5" rot="R180" xref="yes"/>
+</segment>
+<segment>
 <pinref part="X1" gate="G$1" pin="2"/>
 <wire x1="22.86" y1="22.86" x2="27.94" y2="22.86" width="0.1524" layer="91"/>
@@
 <wire x1="86.36" y1="27.94" x2="88.9" y2="27.94" width="0.1524" layer="91"/>
 <label x="88.9" y="27.94" size="1.27" layer="95" ratio="5" xref="yes"/>
-</segment>
-<segment>
-<pinref part="IC2" gate="G$1" pin="D+"/>
-<wire x1="129.54" y1="91.44" x2="121.92" y2="91.44" width="0.1524" layer="91"/>
-<label x="121.92" y="91.44" size="1.27" layer="95" ratio="5" rot="R180" xref="yes"/>
-</segment>
-</net>
-<net name="USB_DN" class="0">
-<segment>
-<pinref part="X1" gate="G$1" pin="3"/>
-<wire x1="22.86" y1="25.4" x2="27.94" y2="25.4" width="0.1524" layer="91"/>
-<label x="27.94" y="25.4" size="1.27" layer="95" ratio="5" xref="yes"/>
-</segment>
-<segment>
-<pinref part="D1" gate="G$1" pin="K_3"/>
-<wire x1="86.36" y1="30.48" x2="88.9" y2="30.48" width="0.1524" layer="91"/>
-<label x="88.9" y="30.48" size="1.27" layer="95" ratio="5" xref="yes"/>
-</segment>
-<segment>
-<pinref part="IC2" gate="G$1" pin="D-"/>
-<wire x1="129.54" y1="88.9" x2="121.92" y2="88.9" width="0.1524" layer="91"/>
-<label x="121.92" y="88.9" size="1.27" layer="95" ratio="5" rot="R180" xref="yes"/>
 </segment>
 </net>
@@
 </segment>
 </net>
+<net name="DTR" class="0">
+<segment>
+<pinref part="IC2" gate="G$1" pin="DTR"/>
+<wire x1="144.78" y1="111.76" x2="144.78" y2="119.38" width="0.1524" layer="91"/>
+<pinref part="C11" gate="G$1" pin="1"/>
+</segment>
+</net>
+<net name="RESET" class="0">
+<segment>
+<pinref part="C11" gate="G$1" pin="2"/>
+<wire x1="144.78" y1="127" x2="144.78" y2="137.16" width="0.1524" layer="91"/>
+<label x="144.78" y="137.16" size="1.27" layer="95" ratio="5" rot="R90" xref="yes"/>
+</segment>
+</net>
