File: electronics/board_template/attiny_44_qfn-24/template_attiny_44.brd (EAGLE design)
At the start: 48 x 48 mm, 17 parts, among them IC2 ATTINY44A-MU, IC3 NCP1117ST50T3G, J1 GROVE_CONNECTOR2.0_1X4, J2 GROVE_CONNECTOR2.0_1X4, J3 10129383-906001ALF, Y1 X322516MLB4SI

Commit message: Fiducials eingefügt
Parts:
- added FID1, FID2, FID3: OPEN-PNP-FIDUCIAL, topo-eng:OPEN-PNP-FIDUCIAL
Changed lines of the file:
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@@
 </element>
 <element name="U$1" library="topo-eng" library_urn="urn:adsk.eagle:library:6646478" package="LOGO_MORPHBOT" value="LOGO_MORPHBOT5MM" x="47.143325" y="1.290628125" smashed="yes" rot="R90"/>
+<element name="FID1" library="topo-eng" library_urn="urn:adsk.eagle:library:6646478" package="OPEN-PNP-FIDUCIAL" value="OPEN-PNP-FIDUCIAL" x="1.623175" y="46.523646875" smashed="yes"/>
+<element name="FID2" library="topo-eng" library_urn="urn:adsk.eagle:library:6646478" package="OPEN-PNP-FIDUCIAL" value="OPEN-PNP-FIDUCIAL" x="46.621534375" y="46.73873125" smashed="yes"/>
+<element name="FID3" library="topo-eng" library_urn="urn:adsk.eagle:library:6646478" package="OPEN-PNP-FIDUCIAL" value="OPEN-PNP-FIDUCIAL" x="1.350690625" y="1.388315625" smashed="yes"/>
 </elements>
 <signals>

Commit message: Logo geändert
Changed lines of the file:
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@@
 <wire x1="15.872465625" y1="39.91308125" x2="4.62865" y2="39.91308125" width="0.5" layer="1"/>
 <wire x1="4.62865" y1="39.91308125" x2="4.04885" y2="40.49288125" width="0.5" layer="1"/>
+<wire x1="44.27974375" y1="40.804375" x2="43.6212625" y2="45.844790625" width="0" layer="19" extent="1-1"/>
+<wire x1="44.279640625" y1="38.866559375" x2="44.27974375" y2="40.804375" width="0" layer="19" extent="1-1"/>
+<wire x1="41.878046875" y1="40.43094375" x2="44.27974375" y2="40.804375" width="0" layer="19" extent="1-1"/>
+<wire x1="40.178046875" y1="38.23094375" x2="41.878046875" y2="40.43094375" width="0" layer="19" extent="1-1"/>
+<wire x1="35.74061875" y1="38.99099375" x2="40.178046875" y2="38.23094375" width="0" layer="19" extent="1-1"/>
+<wire x1="33.526834375" y1="37.8122125" x2="35.140021875" y2="37.731228125" width="0" layer="19" extent="1-1"/>
+<wire x1="35.74061875" y1="40.94099375" x2="35.74061875" y2="38.99099375" width="0" layer="19" extent="1-1"/>
+<wire x1="31.909303125" y1="44.61918125" x2="35.74061875" y2="40.94099375" width="0" layer="19" extent="1-1"/>
+<wire x1="26.94365625" y1="43.29293125" x2="31.909303125" y2="44.61918125" width="0" layer="19" extent="1-1"/>
+<wire x1="26.946446875" y1="39.3299375" x2="26.94365625" y2="43.29293125" width="0" layer="19" extent="1-1"/>
+<wire x1="24.5539375" y1="39.337925" x2="26.946446875" y2="39.3299375" width="0" layer="19" extent="1-1"/>
+<wire x1="20.995678125" y1="35.799090625" x2="24.5539375" y2="39.337925" width="0" layer="19" extent="1-1"/>
+<wire x1="26.54" y1="21.27" x2="26.99033125" y2="12.2144" width="0" layer="19" extent="16-16"/>
 </signal>
 <signal name="SCL">
