File: electronics/board_template/attiny_44_qfn-24/template_attiny_44.sch (EAGLE design)
At the start: 17 parts, among them IC2 ATTINY44A-MU, IC3 NCP1117ST50T3G, J1 GROVE_CONNECTOR2.0_1X4, J2 GROVE_CONNECTOR2.0_1X4, J3 10129383-906001ALF, Y1 X322516MLB4SI

Commit message: Fiducials eingefügt
Parts:
- added FID1, FID2, FID3: OPEN-PNP-FIDUCIAL, topo-eng:OPEN-PNP-FIDUCIAL
Changed lines of the file:
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@@
 <part name="C7" library="rcl" library_urn="urn:adsk.eagle:library:334" deviceset="CPOL-EU" device="C" package3d_urn="urn:adsk.eagle:package:23422/2" value="ST(Semtech) CK1C470M-CRD54 - 47uF"/>
 <part name="U$1" library="topo-eng" library_urn="urn:adsk.eagle:library:6646478" deviceset="LOGO_MORPHBOT" device="5MM"/>
+<part name="FID1" library="topo-eng" library_urn="urn:adsk.eagle:library:6646478" deviceset="OPEN-PNP-FIDUCIAL" device=""/>
+<part name="FID2" library="topo-eng" library_urn="urn:adsk.eagle:library:6646478" deviceset="OPEN-PNP-FIDUCIAL" device=""/>
+<part name="FID3" library="topo-eng" library_urn="urn:adsk.eagle:library:6646478" deviceset="OPEN-PNP-FIDUCIAL" device=""/>
 </parts>
 <sheets>
@@
 </instance>
 <instance part="U$1" gate="G$1" x="88.9" y="2.54" smashed="yes"/>
+<instance part="FID1" gate="FID$1" x="157.48" y="5.08" smashed="yes">
+<attribute name="NAME" x="152.4" y="10.16" size="1.778" layer="94"/>
+</instance>
+<instance part="FID2" gate="FID$1" x="149.86" y="5.08" smashed="yes">
+<attribute name="NAME" x="144.78" y="10.16" size="1.778" layer="94"/>
+</instance>
+<instance part="FID3" gate="FID$1" x="142.24" y="5.08" smashed="yes">
+<attribute name="NAME" x="137.16" y="10.16" size="1.778" layer="94"/>
+</instance>
 </instances>
 <busses>
