File: electronics/board_template/attiny_44_soic-14/template_attiny_44_soic-14.brd (EAGLE design)
At the start: 48 x 48 mm, 17 parts, among them IC1 ATTINY441-SSU, IC3 NCP1117ST50T3G, J1 GROVE_CONNECTOR2.0_1X4, J2 GROVE_CONNECTOR2.0_1X4, J3 10129383-906001ALF, Y1 X322516MLB4SI

Commit message: Fiducials eingefügt
Parts:
- added FID1, FID2, FID3: OPEN-PNP-FIDUCIAL, topo-eng:OPEN-PNP-FIDUCIAL
Changed lines of the file:
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@@
 <attribute name="VALUE" x="35.22874375" y="37.67785625" size="1.27" layer="27" rot="R180" align="center"/>
 </element>
+<element name="FID1" library="topo-eng" library_urn="urn:adsk.eagle:library:6646478" package="OPEN-PNP-FIDUCIAL" value="OPEN-PNP-FIDUCIAL" x="1.47929375" y="1.40814375" smashed="yes"/>
+<element name="FID2" library="topo-eng" library_urn="urn:adsk.eagle:library:6646478" package="OPEN-PNP-FIDUCIAL" value="OPEN-PNP-FIDUCIAL" x="1.662465625" y="46.516315625" smashed="yes"/>
+<element name="FID3" library="topo-eng" library_urn="urn:adsk.eagle:library:6646478" package="OPEN-PNP-FIDUCIAL" value="OPEN-PNP-FIDUCIAL" x="46.355096875" y="46.52634375" smashed="yes"/>
 </elements>
 <signals>

Commit message: Logo geändert
Changed lines of the file:
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@@
 <wire x1="4.62865" y1="39.91308125" x2="4.04885" y2="40.49288125" width="0.5" layer="1"/>
 <contactref element="IC1" pad="14"/>
+<wire x1="44.27974375" y1="40.804375" x2="43.6212625" y2="45.844790625" width="0" layer="19" extent="1-1"/>
+<wire x1="44.279640625" y1="38.866559375" x2="44.27974375" y2="40.804375" width="0" layer="19" extent="1-1"/>
+<wire x1="41.878046875" y1="40.43094375" x2="44.27974375" y2="40.804375" width="0" layer="19" extent="1-1"/>
+<wire x1="40.178046875" y1="38.23094375" x2="41.878046875" y2="40.43094375" width="0" layer="19" extent="1-1"/>
+<wire x1="41.356390625" y1="33.862775" x2="40.178046875" y2="38.23094375" width="0" layer="19" extent="1-1"/>
+<wire x1="32.51774375" y1="33.86785625" x2="40.178046875" y2="38.23094375" width="0" layer="19" extent="1-1"/>
+<wire x1="26.946446875" y1="39.3299375" x2="32.51774375" y2="33.86785625" width="0" layer="19" extent="1-1"/>
+<wire x1="24.5539375" y1="39.337925" x2="26.946446875" y2="39.3299375" width="0" layer="19" extent="1-1"/>
+<wire x1="26.94365625" y1="43.29293125" x2="26.946446875" y2="39.3299375" width="0" layer="19" extent="1-1"/>
+<wire x1="20.995678125" y1="35.799090625" x2="24.5539375" y2="39.337925" width="0" layer="19" extent="1-1"/>
+<wire x1="31.909303125" y1="44.61918125" x2="26.94365625" y2="43.29293125" width="0" layer="19" extent="1-1"/>
+<wire x1="26.54" y1="21.27" x2="26.99033125" y2="12.2144" width="0" layer="19" extent="16-16"/>
 </signal>
 <signal name="SCL">
