File: electronics/board_template/empty_board/template_empty_board.brd (EAGLE design)
At the start: 48 x 48 mm, 13 parts, among them IC3 NCP1117ST50T3G, J1 GROVE_CONNECTOR2.0_1X4, J2 GROVE_CONNECTOR2.0_1X4

Commit message: Logo geändert
Parts:
- IC3: device samacsys:SOT230P700X180-4N@1 -> samacsys:SOT230P700X180-4N
Changed lines of the file:
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@@
 <element name="C2" library="rcl" library_urn="urn:adsk.eagle:library:334" package="PANASONIC_C" package3d_urn="urn:adsk.eagle:package:23422/2" value="ST(Semtech) CK1C470M-CRD54 - 47uF" x="24.89365625" y="43.29293125" smashed="yes" rot="R180">
 <attribute name="NAME" x="24.90483125" y="46.871003125" size="0.8128" layer="25" rot="R180"/>
+<attribute name="POPULARITY" value="4" x="24.89365625" y="43.29293125" size="1.778" layer="27" rot="R180" display="off"/>
 <attribute name="SPICEPREFIX" value="C" x="24.89365625" y="43.29293125" size="1.778" layer="27" rot="R180" display="off"/>
 <attribute name="VALUE" x="27.54365625" y="47.06793125" size="1.016" layer="27" rot="R180"/>
@@
 <element name="C3" library="rcl" library_urn="urn:adsk.eagle:library:334" package="C0603" package3d_urn="urn:adsk.eagle:package:23616/2" value="0603B334K250NT - 330nF" x="4.517928125" y="36.80893125" smashed="yes" rot="R180">
 <attribute name="NAME" x="4.510446875" y="35.626128125" size="0.8128" layer="25" rot="R180"/>
+<attribute name="POPULARITY" value="73" x="4.517928125" y="36.80893125" size="1.778" layer="27" rot="R180" display="off"/>
 <attribute name="SPICEPREFIX" value="C" x="4.517928125" y="36.80893125" size="1.778" layer="27" rot="R180" display="off"/>
 <attribute name="VALUE" x="5.152928125" y="38.71393125" size="1.27" layer="27" rot="R180"/>
@@
 <element name="C1" library="rcl" library_urn="urn:adsk.eagle:library:334" package="C0603" package3d_urn="urn:adsk.eagle:package:23616/2" value="Walsin Tech Corp 0603B104K250CT - 100nF" x="13.74343125" y="39.043334375" smashed="yes">
 <attribute name="NAME" x="13.24070625" y="40.245028125" size="0.8128" layer="25"/>
+<attribute name="POPULARITY" value="73" x="13.74343125" y="39.043334375" size="1.778" layer="27" display="off"/>
 <attribute name="SPICEPREFIX" value="C" x="13.74343125" y="39.043334375" size="1.778" layer="27" display="off"/>
 <attribute name="VALUE" x="13.10843125" y="37.138334375" size="1.27" layer="27"/>
@@
 <attribute name="VALUE" x="18.121734375" y="43.0302875" size="1.27" layer="27" rot="R270"/>
 </element>
-<element name="R1" library="rcl" library_urn="urn:adsk.eagle:library:334" package="R0402" package3d_urn="urn:adsk.eagle:package:23547/2" value="Uniroyal Elec 0402WGF1001TCE - 170R" x="20.000171875" y="44.76161875" smashed="yes" rot="R90">
+<element name="R1" library="rcl" library_urn="urn:adsk.eagle:library:334" package="R0402" package3d_urn="urn:adsk.eagle:package:23547/3" value="Uniroyal Elec 0402WGF1001TCE - 170R" x="20.000171875" y="44.76161875" smashed="yes" rot="R90">
 <attribute name="NAME" x="20.27220625" y="46.072265625" size="0.8128" layer="25" rot="R90"/>
+<attribute name="POPULARITY" value="0" x="20.000171875" y="44.76161875" size="1.778" layer="27" rot="R90" display="off"/>
 <attribute name="SPICEPREFIX" value="R" x="20.000171875" y="44.76161875" size="1.778" layer="27" rot="R90" display="off"/>
 <attribute name="VALUE" x="21.905171875" y="44.12661875" size="1.27" layer="27" rot="R90"/>
 </element>
-<element name="IC3" library="samacsys" package="SOT230P700X180-4N@1" value="NCP1117ST50T3G" x="6.65716875" y="41.91548125" smashed="yes">
+<element name="IC3" library="samacsys" package="SOT230P700X180-4N" value="NCP1117ST50T3G" x="6.65716875" y="41.91548125" smashed="yes">
 <attribute name="ARROW_PART_NUMBER" value="NCP1117ST50T3G" x="6.65716875" y="41.91548125" size="1.778" layer="27" display="off"/>
 <attribute name="ARROW_PRICE-STOCK" value="https://www.arrow.com/en/products/ncp1117st50t3g/on-semiconductor" x="6.65716875" y="41.91548125" size="1.778" layer="27" display="off"/>
@@
 <element name="C7" library="rcl" library_urn="urn:adsk.eagle:library:334" package="PANASONIC_C" package3d_urn="urn:adsk.eagle:package:23422/2" value="ST(Semtech) CK1C470M-CRD54 - 47uF" x="14.96630625" y="43.177225" smashed="yes" rot="R180">
 <attribute name="NAME" x="14.996378125" y="47.0008625" size="0.8128" layer="25" rot="R180"/>
+<attribute name="POPULARITY" value="4" x="14.96630625" y="43.177225" size="1.778" layer="27" rot="R180" display="off"/>
 <attribute name="SPICEPREFIX" value="C" x="14.96630625" y="43.177225" size="1.778" layer="27" rot="R180" display="off"/>
 <attribute name="VALUE" x="17.61630625" y="46.952225" size="1.016" layer="27" rot="R180"/>
@@
 <contactref element="C7" pad="-"/>
 <wire x1="17.01630625" y1="43.177225" x2="16.39966875" y2="43.177225" width="0.5" layer="1"/>
+<wire x1="20.026734375" y1="41.0102875" x2="26.94365625" y2="43.29293125" width="0" layer="19" extent="1-1"/>
+<wire x1="17.01630625" y1="43.177225" x2="20.026734375" y2="41.0102875" width="0" layer="19" extent="1-1"/>
+<wire x1="14.59343125" y1="39.043334375" x2="16.39966875" y2="43.177225" width="0" layer="19" extent="1-1"/>
+<wire x1="20.995678125" y1="35.799090625" x2="20.026734375" y2="41.0102875" width="0" layer="19" extent="1-1"/>
+<wire x1="5.367928125" y1="36.80893125" x2="14.59343125" y2="39.043334375" width="0" layer="19" extent="1-1"/>
+<wire x1="3.25716875" y1="44.21548125" x2="5.367928125" y2="36.80893125" width="0" layer="19" extent="1-1"/>
 </signal>
 <signal name="PC4/SDA">
