File: electronics/boards/tt-motor_driver_and_encoder/tt-motor_driver_and_encoder.brd (EAGLE design)
At the start: 35 x 18 mm, 23 parts, among them IC1 ATTINY441-SSU, IC2 A4953ELJTR-T, IC3 NCP1117ST50T3G, J2 GROVE_CONNECTOR2.0_1X4

Commit message: TT-Motor-Board: Morphbot-Logo entfernt
Parts:
- removed U$1: LOGO_MORPHBOT5MM, topo-eng:LOGO_MORPHBOT
Changed lines of the file:
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@@
 <attribute name="VALUE" x="8.106728125" y="4.636021875" size="1.016" layer="27"/>
 </element>
-<element name="U$1" library="topo-eng" library_urn="urn:adsk.eagle:library:6646478" package="LOGO_MORPHBOT" value="LOGO_MORPHBOT5MM" x="70.857021875" y="32.766421875" smashed="yes" rot="R90"/>
 <element name="IC1" library="samacsys" package="SOIC127P600X175-14N" value="ATTINY441-SSU" x="18.77625" y="13.806096875" smashed="yes" rot="R270">
 <attribute name="ARROW_PART_NUMBER" value="ATTINY441-SSU" x="18.77625" y="13.806096875" size="1.778" layer="27" rot="R270" display="off"/>
