File: electronics/boards/tt-motor_driver_and_encoder/tt-motor_driver_and_encoder.sch (EAGLE design)
At the start: 23 parts, among them IC1 ATTINY441-SSU, IC2 A4953ELJTR-T, IC3 NCP1117ST50T3G, J2 GROVE_CONNECTOR2.0_1X4

Commit message: TT-Motor-Board: Morphbot-Logo entfernt
Parts:
- removed U$1: LOGO_MORPHBOT5MM, topo-eng:LOGO_MORPHBOT5MM
Changed lines of the file:
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@@
 <part name="IC3" library="samacsys" deviceset="NCP1117ST50T3G" device=""/>
 <part name="C7" library="rcl" library_urn="urn:adsk.eagle:library:334" deviceset="CPOL-EU" device="C" package3d_urn="urn:adsk.eagle:package:23422/2" value="ST(Semtech) CK1C470M-CRD54 - 47uF"/>
-<part name="U$1" library="topo-eng" library_urn="urn:adsk.eagle:library:6646478" deviceset="LOGO_MORPHBOT" device="5MM"/>
 <part name="IC1" library="samacsys" deviceset="ATTINY441-SSU" device=""/>
 <part name="FID1" library="topo-eng" library_urn="urn:adsk.eagle:library:6646478" deviceset="OPEN-PNP-FIDUCIAL" device=""/>
@@
 <attribute name="VALUE" x="21.463" y="38.5826" size="1.778" layer="96"/>
 </instance>
-<instance part="U$1" gate="G$1" x="88.9" y="2.54" smashed="yes"/>
 <instance part="IC1" gate="G$1" x="86.36" y="139.7" smashed="yes">
 <attribute name="NAME" x="212.09" y="147.32" size="1.778" layer="95" align="center-left"/>
