File: electronics/board_template/ESP32/template_esp32.brd (EAGLE design)
At the start: 48 x 48 mm, 55 parts, among them IC1 ESP-WROOM-32D, IC2 CP2104-F03-GMR, IC3 NCP1117ST50T3G, IC4 LMV358IDGKRG4, IC5 NCP1117ST33T3G, J1 GROVE_CONNECTOR2.0_1X4, J2 GROVE_CONNECTOR2.0_1X4, J4 10129383-912001ALF, J5 10129383-912001ALF, Q1 FDN340P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

Commit message: Logo geändert
Parts:
- moved U$1 0.30 mm to (0.37, 44.9)
Changed lines of the file:
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@@
 <attribute name="VALUE" x="13.968846875" y="29.92159375" size="1.27" layer="27" rot="R270"/>
 </element>
-<element name="U$1" library="topo-eng" library_urn="urn:adsk.eagle:library:6646478" package="LOGO_MOPRHBOT_3MM" value="LOGO_MORPHBOT3MM" x="0.088325" y="44.75038125" smashed="yes"/>
+<element name="U$1" library="topo-eng" library_urn="urn:adsk.eagle:library:6646478" package="LOGO_MOPRHBOT_3MM" value="LOGO_MORPHBOT3MM" x="0.370340625" y="44.85108125" smashed="yes"/>
 <element name="FID1" library="topo-eng" library_urn="urn:adsk.eagle:library:6646478" package="OPEN-PNP-FIDUCIAL" value="OPEN-PNP-FIDUCIAL" x="2.252828125" y="2.971290625" smashed="yes"/>
 <element name="FID2" library="topo-eng" library_urn="urn:adsk.eagle:library:6646478" package="OPEN-PNP-FIDUCIAL" value="OPEN-PNP-FIDUCIAL" x="37.827975" y="2.543028125" smashed="yes"/>
@@
 <via x="9.33243125" y="7.1559875" extent="1-16" drill="0.35"/>
 <via x="1.511059375" y="19.693871875" extent="1-16" drill="0.35"/>
+<wire x1="32.347753125" y1="38.699390625" x2="39.847753125" y2="46.199390625" width="0" layer="19" extent="1-1"/>
+<wire x1="22.337753125" y1="43.414390625" x2="32.347753125" y2="38.699390625" width="0" layer="19" extent="1-1"/>
+<wire x1="17.476159375" y1="41.516775" x2="22.337753125" y2="43.414390625" width="0" layer="19" extent="1-1"/>
+<wire x1="13.320940625" y1="38.2025625" x2="13.2708375" y2="38.404578125" width="0" layer="19" extent="1-1"/>
+<wire x1="11.34494375" y1="34.79154375" x2="13.320940625" y2="38.2025625" width="0" layer="19" extent="1-1"/>
+<wire x1="11.348" y1="32.664671875" x2="11.34494375" y2="34.79154375" width="0" layer="19" extent="1-1"/>
+<wire x1="12.52669375" y1="32.74525" x2="11.348" y2="32.664671875" width="0" layer="19" extent="1-1"/>
+<wire x1="12.990128125" y1="29.085625" x2="12.52669375" y2="32.74525" width="0" layer="19" extent="1-1"/>
+<wire x1="17.2094" y1="30.17795" x2="12.990128125" y2="29.085625" width="0" layer="19" extent="1-1"/>
+<wire x1="17.55955" y1="34.154646875" x2="17.2094" y2="30.17795" width="0" layer="19" extent="1-1"/>
+<wire x1="14.3081" y1="44.9694375" x2="17.476159375" y2="41.516775" width="0" layer="19" extent="1-1"/>
+<wire x1="11.525746875" y1="44.94625625" x2="14.3081" y2="44.9694375" width="0" layer="19" extent="1-1"/>
+<wire x1="6.319678125" y1="34.305984375" x2="11.34494375" y2="34.79154375" width="0" layer="19" extent="1-1"/>
+<wire x1="4.804853125" y1="30.67039375" x2="6.319678125" y2="34.305984375" width="0" layer="19" extent="1-1"/>
+<wire x1="3.281409375" y1="37.36804375" x2="6.319678125" y2="34.305984375" width="0" layer="19" extent="1-1"/>
+<wire x1="1.919678125" y1="34.305984375" x2="3.281409375" y2="37.36804375" width="0" layer="19" extent="1-1"/>
+<wire x1="20.19" y1="24.73" x2="17.2094" y2="30.17795" width="0" layer="19" extent="1-1"/>
+<wire x1="20.19" y1="19.27" x2="20.19" y2="24.73" width="0" layer="19" extent="1-1"/>
+<wire x1="3.25716875" y1="44.21548125" x2="3.281409375" y2="37.36804375" width="0" layer="19" extent="1-1"/>
+<wire x1="16.270371875" y1="12.997915625" x2="20.19" y2="19.27" width="0" layer="19" extent="1-1"/>
+<wire x1="11.1113625" y1="12.720253125" x2="16.270371875" y2="12.997915625" width="0" layer="19" extent="1-1"/>
+<wire x1="20.19" y1="8.73" x2="16.270371875" y2="12.997915625" width="0" layer="19" extent="1-1"/>
+<wire x1="20.19" y1="3.27" x2="20.19" y2="8.73" width="0" layer="19" extent="1-1"/>
+<wire x1="23.4645875" y1="1.3874875" x2="20.19" y2="3.27" width="0" layer="19" extent="1-16"/>
+<wire x1="30.127871875" y1="13.56601875" x2="26.99033125" y2="12.2144" width="0" layer="19" extent="1-1"/>
+<wire x1="30.336665625" y1="15.207075" x2="30.127871875" y2="13.56601875" width="0" layer="19" extent="1-1"/>
+<wire x1="33.69586875" y1="17.84271875" x2="30.336665625" y2="15.207075" width="0" layer="19" extent="1-1"/>
+<wire x1="39.1917" y1="19.484865625" x2="33.69586875" y2="17.84271875" width="0" layer="19" extent="1-1"/>
+<wire x1="40.860321875" y1="22.243528125" x2="39.1917" y2="19.484865625" width="0" layer="19" extent="1-1"/>
+<wire x1="39.23296875" y1="26.0091375" x2="40.860321875" y2="22.243528125" width="0" layer="19" extent="1-1"/>
+<wire x1="36.12831875" y1="25.24850625" x2="39.23296875" y2="26.0091375" width="0" layer="19" extent="1-1"/>
+<wire x1="39.847753125" y1="29.199390625" x2="39.23296875" y2="26.0091375" width="0" layer="19" extent="1-1"/>
+<wire x1="45.1917" y1="19.484865625" x2="40.860321875" y2="22.243528125" width="0" layer="19" extent="1-1"/>
+<wire x1="45.23296875" y1="26.0091375" x2="40.860321875" y2="22.243528125" width="0" layer="19" extent="1-1"/>
+<wire x1="9.33243125" y1="7.1559875" x2="11.1113625" y2="12.720253125" width="0" layer="19" extent="1-1"/>
+<wire x1="7.72095625" y1="5.80261875" x2="9.33243125" y2="7.1559875" width="0" layer="19" extent="1-1"/>
+<wire x1="5.787378125" y1="4.49425625" x2="7.72095625" y2="5.80261875" width="0" layer="19" extent="1-1"/>
+<wire x1="3.2976375" y1="8.655196875" x2="5.787378125" y2="4.49425625" width="0" layer="19" extent="1-1"/>
+<wire x1="3.864046875" y1="13.236940625" x2="3.2976375" y2="8.655196875" width="0" layer="19" extent="1-1"/>
+<wire x1="4.6066375" y1="16.04546875" x2="2.764384375" y2="14.42755625" width="0" layer="19" extent="1-1"/>
+<wire x1="4.605353125" y1="17.2899625" x2="4.6066375" y2="16.04546875" width="0" layer="19" extent="1-1"/>
+<wire x1="1.511059375" y1="19.693871875" x2="4.605353125" y2="17.2899625" width="0" layer="19" extent="1-1"/>
+<wire x1="8.75" y1="22.4" x2="4.605353125" y2="17.2899625" width="0" layer="19" extent="1-1"/>
+<wire x1="40.36744375" y1="12.7683" x2="39.1917" y2="19.484865625" width="0" layer="19" extent="1-1"/>
+<wire x1="42.623328125" y1="13.10056875" x2="40.36744375" y2="12.7683" width="0" layer="19" extent="1-1"/>
+<wire x1="44.93733125" y1="8.989084375" x2="42.623328125" y2="13.10056875" width="0" layer="19" extent="1-1"/>
+<wire x1="35.931128125" y1="8.635440625" x2="40.36744375" y2="12.7683" width="0" layer="19" extent="1-1"/>
 </signal>
 <signal name="SDA">
