File: electronics/boards/Stromversorgung/stromversorgung.brd (EAGLE design)
At the start: 48 x 48 mm, 13 parts, among them IC2 NCP1117ST33T3G, J1 GROVE_CONNECTOR2.0_1X4, J2 GROVE_CONNECTOR2.0_1X4, J3 GROVE_CONNECTOR2.0_1X4, J4 GROVE_CONNECTOR2.0_1X4

Commit message: Template Empty Board an anderen Linearregler angepasst
Routing:
- net GND: track 131.4 -> 119.4 mm
Changed lines of the file:
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@@
 <vertex x="47" y="0"/>
 </polygon>
-<wire x1="14.646834375" y1="35.799090625" x2="20.995678125" y2="35.799090625" width="0.5" layer="1"/>
-<wire x1="10.608078125" y1="39.837846875" x2="14.646834375" y2="35.799090625" width="0.5" layer="1"/>
 <contactref element="IC2" pad="1"/>
 <contactref element="C1" pad="2"/>

Commit message: Logo hinzugefügt
Parts:
- added U$1: LOGO_MORPHBOT5MM, topo-eng:LOGO_MORPHBOT
Changed lines of the file:
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@@
 <layer number="104" name="Name" color="7" fill="1" visible="no" active="yes"/>
 <layer number="116" name="Patch_BOT" color="9" fill="4" visible="no" active="yes"/>
+<layer number="120" name="brd_placement_notes" color="7" fill="1" visible="yes" active="yes"/>
 <layer number="121" name="_tsilk" color="7" fill="1" visible="no" active="yes"/>
 <layer number="122" name="_bsilk" color="7" fill="1" visible="no" active="yes"/>
+<layer number="144" name="DrillLegend" color="7" fill="1" visible="yes" active="yes"/>
+<layer number="145" name="DrillLegend_01-16" color="7" fill="1" visible="yes" active="yes"/>
+<layer number="146" name="DrillLegend_01-20" color="7" fill="1" visible="yes" active="yes"/>
 <layer number="151" name="HeatSink" color="14" fill="1" visible="no" active="no"/>
+<layer number="198" name="BMP198" color="7" fill="1" visible="yes" active="yes"/>
+<layer number="199" name="Contour" color="7" fill="1" visible="yes" active="yes"/>
 <layer number="200" name="200bmp" color="1" fill="10" visible="no" active="no"/>
 <layer number="201" name="201bmp" color="2" fill="1" visible="no" active="no"/>
@@
 <layer number="207" name="207bmp" color="15" fill="10" visible="no" active="no"/>
 <layer number="208" name="208bmp" color="9" fill="10" visible="no" active="yes"/>
+<layer number="209" name="Route9Document" color="7" fill="1" visible="yes" active="yes"/>
+<layer number="210" name="Route10Document" color="7" fill="1" visible="yes" active="yes"/>
+<layer number="211" name="Route11Document" color="7" fill="1" visible="yes" active="yes"/>
+<layer number="212" name="Route12Document" color="7" fill="1" visible="yes" active="yes"/>
+<layer number="213" name="Route13Document" color="7" fill="1" visible="yes" active="yes"/>
+<layer number="214" name="Route14Document" color="7" fill="1" visible="yes" active="yes"/>
+<layer number="215" name="Route15Document" color="7" fill="1" visible="yes" active="yes"/>
+<layer number="216" name="BottomDocument" color="7" fill="1" visible="yes" active="yes"/>
+<layer number="220" name="DimensionDocument" color="7" fill="1" visible="yes" active="yes"/>
+<layer number="221" name="tPlaceDocument" color="7" fill="1" visible="yes" active="yes"/>
+<layer number="222" name="bPlaceDocument" color="7" fill="1" visible="yes" active="yes"/>
+<layer number="225" name="tNamesDocument" color="7" fill="1" visible="yes" active="yes"/>
+<layer number="226" name="bNamesDocument" color="7" fill="1" visible="yes" active="yes"/>
+<layer number="227" name="tValuesDocument" color="7" fill="1" visible="yes" active="yes"/>
+<layer number="228" name="bValuesDocument" color="7" fill="1" visible="yes" active="yes"/>
+<layer number="229" name="tStopDocument" color="7" fill="1" visible="yes" active="yes"/>
+<layer number="230" name="bStopDocument" color="7" fill="1" visible="yes" active="yes"/>
+<layer number="231" name="tCreamDocument" color="7" fill="1" visible="yes" active="yes"/>
+<layer number="232" name="bCreamDocument" color="7" fill="1" visible="yes" active="yes"/>
+<layer number="233" name="tFinishDocument" color="7" fill="1" visible="yes" active="yes"/>
+<layer number="234" name="bFinishDocument" color="7" fill="1" visible="yes" active="yes"/>
+<layer number="235" name="tGlueDocument" color="7" fill="1" visible="yes" active="yes"/>
+<layer number="236" name="bGlueDocument" color="7" fill="1" visible="yes" active="yes"/>
+<layer number="244" name="DrillsDocument" color="7" fill="1" visible="yes" active="yes"/>
+<layer number="245" name="HolesDocument" color="7" fill="1" visible="yes" active="yes"/>
+<layer number="246" name="MillingDocument" color="7" fill="1" visible="yes" active="yes"/>
+<layer number="247" name="MeasuresDocument" color="7" fill="1" visible="yes" active="yes"/>
 <layer number="250" name="Descript" color="3" fill="1" visible="no" active="no"/>
 <layer number="251" name="SMDround" color="12" fill="11" visible="no" active="no"/>
@@
 <attribute name="NAME" x="38.517871875" y="28.62524375" size="0.8128" layer="25" font="vector" ratio="10" rot="R270"/>
 </element>
+<element name="U$1" library="topo-eng" library_urn="urn:adsk.eagle:library:6646478" package="LOGO_MORPHBOT" value="LOGO_MORPHBOT5MM" x="47.4088375" y="0.643234375" smashed="yes" rot="R90"/>
 </elements>
 <signals>

Commit message: Fiducials eingefügt
Parts:
- added FID1, FID2, FID3: OPEN-PNP-FIDUCIAL, topo-eng:OPEN-PNP-FIDUCIAL
Changed lines of the file:
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@@
 </element>
 <element name="U$1" library="topo-eng" library_urn="urn:adsk.eagle:library:6646478" package="LOGO_MORPHBOT" value="LOGO_MORPHBOT5MM" x="47.4088375" y="0.643234375" smashed="yes" rot="R90"/>
+<element name="FID1" library="topo-eng" library_urn="urn:adsk.eagle:library:6646478" package="OPEN-PNP-FIDUCIAL" value="OPEN-PNP-FIDUCIAL" x="1.504975" y="1.555090625" smashed="yes"/>
+<element name="FID2" library="topo-eng" library_urn="urn:adsk.eagle:library:6646478" package="OPEN-PNP-FIDUCIAL" value="OPEN-PNP-FIDUCIAL" x="1.4136625" y="46.701515625" smashed="yes"/>
+<element name="FID3" library="topo-eng" library_urn="urn:adsk.eagle:library:6646478" package="OPEN-PNP-FIDUCIAL" value="OPEN-PNP-FIDUCIAL" x="46.340315625" y="46.51664375" smashed="yes"/>
 </elements>
 <signals>

Commit message: Logo geändert
Changed lines of the file:
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@@
 <contactref element="J3" pad="4"/>
 <contactref element="J4" pad="4"/>
+<wire x1="30.67439375" y1="41.061465625" x2="37.036471875" y2="43.275090625" width="0" layer="19" extent="1-1"/>
+<wire x1="26.946446875" y1="39.3299375" x2="30.67439375" y2="41.061465625" width="0" layer="19" extent="1-1"/>
+<wire x1="24.5539375" y1="39.337925" x2="26.946446875" y2="39.3299375" width="0" layer="19" extent="1-1"/>
+<wire x1="26.94365625" y1="43.29293125" x2="26.946446875" y2="39.3299375" width="0" layer="19" extent="1-1"/>
+<wire x1="20.995678125" y1="35.799090625" x2="24.5539375" y2="39.337925" width="0" layer="19" extent="1-1"/>
+<wire x1="24.417228125" y1="26.3678125" x2="20.995678125" y2="35.799090625" width="0" layer="19" extent="1-1"/>
+<wire x1="12.35263125" y1="27.084246875" x2="24.417228125" y2="26.3678125" width="0" layer="19" extent="1-1"/>
+<wire x1="35.936871875" y1="20.68824375" x2="26.99033125" y2="12.2144" width="0" layer="19" extent="1-1"/>
 </signal>
 <signal name="SCL">
